File: PENIS.sch (KiCad schematic (older format))
At the start: 327 parts

Commit message: 2
Parts:
- removed C?: 4.7nF, symbol Device:C_Small
- removed C?: 100nF, symbol Device:C_Small
- removed D?: SMF 9.0CA, symbol Device:D_TVS
- removed D?: WS2812B, LED_SMD:LED_WS2812B_PLCC4_5.0x5.0mm_P3.2mm, symbol LED:WS2812B
- removed F?: Polyfuse_Small, symbol Device:Polyfuse_Small
- removed J?: USB_C_Receptacle_USB2.0, symbol Connector:USB_C_Receptacle_USB2.0
- removed R?: 1M, symbol Device:R_Small
- removed R? (x2): 5.1k, symbol Device:R_Small
- added C104, C107, C110, C112, C113, C114, C115, C15, C16, C17, C23, C30, C31, C38, C39, C40, C46, C47, C53, C6, C61, C69, C7, C75, C8, C81, C87, C9, C92, C93, C99: 100nF, Capacitor_SMD:C_0805_2012Metric, symbol Device:C_Small
- added D103, D125, D141, D15, D155, D16, D17, D176, D185, D199, D200, D23, D24, D25, D31, D32, D33, D39, D40, D41, D47, D48, D54, D6, D62, D68, D7, D74, D8, D85, D9: WS2812B, LED_SMD:LED_WS2812B_PLCC4_5.0x5.0mm_P3.2mm, symbol LED:WS2812B
- added D104, D110, D121, D126, D134, D142, D147, D156, D162, D168, D177, D186, D190, D195, D75, D87, D93: 1n4148, Diode_THT:D_DO-35_SOD27_P10.16mm_Horizontal, symbol Device:D_Small
- added F1: 500mA, Fuse:Fuse_1206_3216Metric, symbol Device:Polyfuse_Small
- added J2: Conn_01x04_Female, Connector_PinSocket_2.54mm:PinSocket_1x04_P2.54mm_Vertical, symbol Connector:Conn_01x04_Female
- added MX1, MX12, MX17, MX23, MX28, MX33, MX39, MX44, MX49, MX55, MX6, MX61, MX67, MX73, MX80, MX84, MX89: MX-NoLED, MX_Only:MXOnly-1U-Hotswap, symbol MX_Alps_Hybrid:MX-NoLED
- added P1: USB_C_Plug, Connector_USB:USB_C_Receptacle_HRO_TYPE-C-31-M-12, symbol Connector:USB_C_Plug
- added R1: 5.1k, Resistor_SMD:R_0805_2012Metric, symbol Device:R_Small
- added U2: USBLC6-2SC6, Package_TO_SOT_SMD:SOT-23-6, symbol Power_Protection:USBLC6-2SC6
- C1, C10, C100, C101, C102, C103, C105, C106, C108, C109, C11, C111, C12, C13, C14, C19, C2, C20, C21, C22, C24, C25, C26, C27, C28, C29, C3, C32, C33, C34, C35, C36, C37, C4, C41, C42, C43, C44, C45, C48, C49, C5, C50, C51, C52, C54, C55, C56, C57, C58, C59, C60, C62, C63, C64, C65, C66, C67, C68, C70, C71, C72, C73, C74, C76, C77, C78, C79, C80, C82, C83, C84, C85, C86, C88, C89, C90, C91, C94, C95, C96, C97, C98: renamed from C?; footprint (none) -> Capacitor_SMD:C_0805_2012Metric
- C18: renamed from C?; value C_Small -> 100nF; footprint (none) -> Capacitor_SMD:C_0805_2012Metric
- D105, D106, D107, D108, D109, D111, D112, D113, D114, D118, D119, D120, D122, D127, D128, D129, D130, D131, D135, D136, D137, D138, D143, D144, D145, D146, D148, D149, D150, D151, D152, D157, D158, D159, D160, D161, D163, D164, D165, D166, D167, D169, D170, D171, D172, D173, D178, D179, D180, D181, D183, D184, D187, D188, D189, D191, D192, D193, D194, D196, D197, D198, D76, D77, D78, D79, D86, D88, D89, D90, D91, D92, D94, D95, D96, D97: renamed from D?; footprint (none) -> Diode_THT:D_DO-35_SOD27_P10.16mm_Horizontal
- D55: renamed from D?; value D_Small -> 1n4148; footprint (none) -> Diode_THT:D_DO-35_SOD27_P10.16mm_Horizontal
- D56: renamed from D?; footprint (none) -> Diode_SMD:D_SOD-123
- MX10, MX76: renamed from MX?; footprint (none) -> MX_Only:MXOnly-2.25U-Hotswap
- MX11, MX16, MX22, MX54, MX60, MX66, MX72: renamed from MX?; footprint (none) -> MX_Only:MXOnly-1.25U-Hotswap
- MX13, MX14, MX15, MX18, MX19, MX2, MX20, MX21, MX24, MX25, MX26, MX27, MX29, MX3, MX30, MX31, MX32, MX34, MX35, MX36, MX37, MX4, MX40, MX41, MX42, MX43, MX45, MX46, MX47, MX48, MX5, MX50, MX51, MX52, MX53, MX56, MX57, MX58, MX59, MX62, MX63, MX64, MX65, MX68, MX69, MX7, MX70, MX71, MX74, MX75, MX81, MX82, MX83, MX85, MX86, MX87, MX88, MX90, MX91, MX92: renamed from MX?; footprint (none) -> MX_Only:MXOnly-1U-Hotswap
- MX38: renamed from MX?; footprint (none) -> MX_Only:MXOnly-6.25U-Hotswap
- MX77: renamed from MX?; footprint (none) -> MX_Only:MXOnly-2.75U-Hotswap
- MX78: renamed from MX?; footprint (none) -> MX_Only:MXOnly-2U-Hotswap
- MX79, MX8: renamed from MX?; footprint (none) -> MX_Only:MXOnly-1.5U-Hotswap
- MX9: renamed from MX?; footprint (none) -> MX_Only:MXOnly-1.75U-Hotswap
- Q1: renamed from Q?; footprint (none) -> keyboard_parts_1:SOT23-3_HSOL
- R3, R4, R5: renamed from R?; footprint (none) -> Resistor_SMD:R_0805_2012Metric
- SW1: renamed from SW?; footprint (none) -> Button_Switch_THT:SW_PUSH_6mm
- SW2: renamed from SW?; footprint (none) -> Rotary_Encoder:RotaryEncoder_Alps_EC11E-Switch_Vertical_H20mm
- gave numbers to parts that had none: 75
Connections:
- net +3V3: now also U1.1 (VBAT)
- net +5V: now also C104.1, C107.1, C110.1, C112.1, C113.1, C114.1, C115.1, C15.1, C16.1, C17.1, C23.1, C30.1, C31.1, C38.1, C39.1, C40.1, C46.1, C47.1, C53.1, C6.1, C61.1, C69.1, C7.1, C75.1, C8.1, C81.1, C87.1, C9.1, C92.1, C93.1, C99.1, D103.1 (VDD), D125.1 (VDD), D141.1 (VDD), D15.1 (VDD), D155.1 (VDD), D16.1 (VDD), D17.1 (VDD), D176.1 (VDD), D185.1 (VDD), D199.1 (VDD), D200.1 (VDD), D23.1 (VDD), D24.1 (VDD), D25.1 (VDD), D31.1 (VDD), D32.1 (VDD), D33.1 (VDD), D39.1 (VDD), D40.1 (VDD), D41.1 (VDD), D47.1 (VDD), D48.1 (VDD), D54.1 (VDD), D6.1 (VDD), D62.1 (VDD), D68.1 (VDD), D7.1 (VDD), D74.1 (VDD), D8.1 (VDD), D85.1 (VDD), D9.1 (VDD), F1.1, J2.3 (Pin_3), U2.5 (VBUS)
- net COL0: now also MX1.1 (COL)
- net COL1: now also MX6.1 (COL)
- net COL10: now also MX55.1 (COL)
- net COL11: now also MX61.1 (COL)
- net COL12: now also MX67.1 (COL)
- net COL13: now also MX73.1 (COL)
- net COL15: now also MX80.1 (COL)
- net COL16: now also MX84.1 (COL)
- net COL17: now also MX89.1 (COL)
- net COL2: now also MX12.1 (COL)
- net COL3: now also MX17.1 (COL)
- net COL4: now also MX23.1 (COL)
- net COL5: now also MX28.1 (COL)
- net COL6: now also MX34.1 (COL), MX33.1 (COL)
- net COL7: now also MX39.1 (COL)
- net COL8: now also MX44.1 (COL)
- net COL9: now also MX49.1 (COL)
- net D+: now also U2.4 (I/O2)
- net D-: now also U2.6 (I/O1)
- net GND: now also C104.2, C107.2, C110.2, C112.2, C113.2, C114.2, C115.2, C15.2, C16.2, C17.2, C23.2, C30.2, C31.2, C38.2, C39.2, C40.2, C46.2, C47.2, C53.2, C6.2, C61.2, C69.2, C7.2, C75.2, C8.2, C81.2, C87.2, C9.2, C92.2, C93.2, C99.2, D103.3 (VSS), D125.3 (VSS), D141.3 (VSS), D15.3 (VSS), D155.3 (VSS), D16.3 (VSS), D17.3 (VSS), D176.3 (VSS), D185.3 (VSS), D199.3 (VSS), D200.3 (VSS), D23.3 (VSS), D24.3 (VSS), D25.3 (VSS), D31.3 (VSS), D32.3 (VSS), D33.3 (VSS), D39.3 (VSS), D40.3 (VSS), D41.3 (VSS), D47.3 (VSS), D48.3 (VSS), D54.3 (VSS), D6.3 (VSS), D62.3 (VSS), D68.3 (VSS), D7.3 (VSS), D74.3 (VSS), D8.3 (VSS), D85.3 (VSS), D9.3 (VSS), J2.4 (Pin_4), P1.A1 (GND), P1.A12 (GND), P1.B1 (GND), P1.B12 (GND), P1.S1 (SHIELD), R1.1, U2.2 (GND)
- net ROW0: now also D86.1 (K), D104.1 (K), D110.1 (K), D121.1 (K), D126.1 (K), D134.1 (K), D142.1 (K), D147.1 (K), D156.1 (K), D162.1 (K), D168.1 (K), D177.1 (K), D186.1 (K), D190.1 (K), D195.1 (K), D87.1 (K), D93.1 (K)
- net ROW1: now also D105.1 (K), D111.1 (K), D122.1 (K), D135.1 (K), D143.1 (K), D148.1 (K), D157.1 (K), D163.1 (K), D169.1 (K), D178.1 (K), D183.1 (K), D187.1 (K), D191.1 (K), D196.1 (K), D88.1 (K), D94.1 (K), D75.1 (K); no longer D106.1 (K), D112.1 (K), D118.1 (K), D128.1 (K), D136.1 (K), D144.1 (K), D149.1 (K), D158.1 (K), D164.1 (K), D170.1 (K), D179.1 (K), D188.1 (K), D192.1 (K), D197.1 (K), D76.1 (K), D89.1 (K), D95.1 (K)
- net ROW2: now also D106.1 (K), D112.1 (K), D118.1 (K), D128.1 (K), D136.1 (K), D144.1 (K), D149.1 (K), D158.1 (K), D164.1 (K), D170.1 (K), D179.1 (K), D184.1 (K), D188.1 (K), D192.1 (K), D197.1 (K), D76.1 (K), D89.1 (K), D95.1 (K); no longer D107.1 (K), D113.1 (K), D119.1 (K), D129.1 (K), D137.1 (K), D145.1 (K), D150.1 (K), D159.1 (K), D165.1 (K), D171.1 (K), D180.1 (K), D77.1 (K), D90.1 (K), D96.1 (K)
- net ROW3: now also D107.1 (K), D113.1 (K), D119.1 (K), D129.1 (K), D137.1 (K), D145.1 (K), D150.1 (K), D159.1 (K), D165.1 (K), D171.1 (K), D180.1 (K), D77.1 (K), D90.1 (K), D96.1 (K); no longer D108.1 (K), D114.1 (K), D120.1 (K), D130.1 (K), D138.1 (K), D146.1 (K), D151.1 (K), D160.1 (K), D166.1 (K), D172.1 (K), D181.1 (K), D193.1 (K), D78.1 (K), D91.1 (K)
- net ROW4: now also D108.1 (K), D114.1 (K), D120.1 (K), D130.1 (K), D138.1 (K), D146.1 (K), D151.1 (K), D160.1 (K), D166.1 (K), D172.1 (K), D181.1 (K), D193.1 (K), D78.1 (K), D91.1 (K); no longer D109.1 (K), D131.1 (K), D152.1 (K), D161.1 (K), D167.1 (K), D173.1 (K), D189.1 (K), D194.1 (K), D198.1 (K), D79.1 (K), D92.1 (K), D97.1 (K)
- net SCL: now also J2.2 (Pin_2)
- net SDA: now also J2.1 (Pin_1)
- net VCC: now also F1.2, P1.A4 (VBUS), P1.A9 (VBUS), P1.B4 (VBUS), P1.B9 (VBUS)
- net WS2812C_2: now reaches U1.29 (PA8)
- net WS2812C_2: now also D7.4 (DIN)
- net ROW5: now reaches U1.38 (PA15)
- net ROW5: now also D109.1 (K), D131.1 (K), D152.1 (K), D161.1 (K), D167.1 (K), D173.1 (K), D189.1 (K), D194.1 (K), D198.1 (K), D79.1 (K), D92.1 (K), D97.1 (K)
- net at D84.2 (DOUT): now also D117.4 (DIN)
- removed net WC2812C: D117.2 (DOUT), D132.2 (DOUT), D133.2 (DOUT), D174.2 (DOUT), D182.2 (DOUT)
- removed net WS2812C: D1.4 (DIN), D2.4 (DIN), D3.4 (DIN), D4.4 (DIN), D5.4 (DIN), U1.28 (PB15)
- new net: D16.4 (DIN), D8.2 (DOUT)
- new net: D7.2 (DOUT), D8.4 (DIN)
- new net: D16.2 (DOUT), D24.4 (DIN)
- new net: D24.2 (DOUT), D32.4 (DIN)
- new net: D32.2 (DOUT), D40.4 (DIN)
- new net: D40.2 (DOUT), D9.4 (DIN)
- new net: D17.4 (DIN), D9.2 (DOUT)
- new net: D17.2 (DOUT), D25.4 (DIN)
- new net: D25.2 (DOUT), D33.4 (DIN)
- new net: D33.2 (DOUT), D41.4 (DIN)
- new net: D41.2 (DOUT), D48.4 (DIN)
- new net: D199.2 (DOUT), D2.4 (DIN)
- new net: D185.2 (DOUT), D199.4 (DIN)
- new net: D75.2 (A), MX1.2 (ROW)
- new net: D174.2 (DOUT), D6.4 (DIN)
- new net: D87.2 (A), MX6.2 (ROW)
- new net: D93.2 (A), MX12.2 (ROW)
- new net: D104.2 (A), MX17.2 (ROW)
- new net: D110.2 (A), MX23.2 (ROW)
- new net: D121.2 (A), MX28.2 (ROW)
- new net: D134.2 (A), MX39.2 (ROW)
- new net: D142.2 (A), MX44.2 (ROW)
- new net: D147.2 (A), MX49.2 (ROW)
- new net: D156.2 (A), MX55.2 (ROW)
- new net: D162.2 (A), MX61.2 (ROW)
- new net: D168.2 (A), MX67.2 (ROW)
- new net: D177.2 (A), MX73.2 (ROW)
- new net: D126.2 (A), MX33.2 (ROW)
- new net: D200.2 (DOUT), D3.4 (DIN)
- new net: D182.2 (DOUT), D200.4 (DIN)
- new net: D132.2 (DOUT), D4.4 (DIN)
- new net: D133.2 (DOUT), D5.4 (DIN)
- new net: P1.A5 (CC), R1.2
- new net: P1.A6 (D+), U2.3 (I/O2)
- new net: P1.A7 (D-), U2.1 (I/O1)
- new net: D186.2 (A), MX80.2 (ROW)
- new net: D190.2 (A), MX84.2 (ROW)
- new net: D195.2 (A), MX89.2 (ROW)
- new net: D15.4 (DIN), D6.2 (DOUT)
- new net: D15.2 (DOUT), D23.4 (DIN)
- new net: D23.2 (DOUT), D31.4 (DIN)
- new net: D31.2 (DOUT), D39.4 (DIN)
- new net: D39.2 (DOUT), D47.4 (DIN)
- new net: D47.2 (DOUT), D54.4 (DIN)
- new net: D54.2 (DOUT), D62.4 (DIN)
- new net: D62.2 (DOUT), D68.4 (DIN)
- new net: D68.2 (DOUT), D74.4 (DIN)
- new net: D74.2 (DOUT), D85.4 (DIN)
- new net: D103.4 (DIN), D85.2 (DOUT)
- new net: D103.2 (DOUT), D125.4 (DIN)
- new net: D125.2 (DOUT), D141.4 (DIN)
- new net: D141.2 (DOUT), D155.4 (DIN)
- new net: D155.2 (DOUT), D176.4 (DIN)
- new net: D176.2 (DOUT), D185.4 (DIN)
- new net WS2812C_1: D1.4 (DIN), U1.28 (PB15)
- no-connect marks 2 -> 13
Other:
- note added: "OLED"
- note added: "RGB Backlight"
- note removed: "USB-C"
- moved on the sheet: C1, C10, C102, C105, C108, C18, C24, C25, C26, C27, C28, C29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

Commit message: MK2: dual layer and shittier in every other way
Parts:
- removed C115, C16, C17, C30, C31, C39, C40, C47, C7, C8, C9, C92: 100nF, Capacitor_SMD:C_0805_2012Metric, symbol Device:C_Small
- removed D16, D17, D24, D25, D32, D33, D40, D41, D48, D7, D8, D9: WS2812B, LED_SMD:LED_WS2812B_PLCC4_5.0x5.0mm_P3.2mm, symbol LED:WS2812B
- D1, D10, D100, D101, D103, D11, D115, D116, D117, D12, D123, D124, D125, D13, D132, D133, D139, D14, D140, D141, D15, D153, D154, D155, D174, D175, D176, D18, D182, D185, D19, D199, D2, D20, D200, D21, D22, D23, D26, D27, D28, D29, D3, D30, D31, D34, D35, D36, D37, D38, D39, D4, D42, D43, D44, D45, D46, D47, D49, D5, D50, D51, D52, D53, D54, D57, D58, D59, D6, D60, D61, D62, D63, D64, D65, D66, D67, D68, D69, D70, D71, D72, D73, D74, D80, D81, D82, D83, D84, D85, D98, D99: footprint LED_SMD:LED_WS2812B_PLCC4_5.0x5.0mm_P3.2mm -> sk6812 mini-e:SK6812MINIE
- D104, D105, D106, D107, D108, D109, D110, D111, D112, D113, D114, D118, D119, D120, D121, D122, D126, D127, D128, D129, D130, D131, D134, D135, D136, D137, D138, D142, D143, D144, D145, D146, D147, D148, D149, D150, D151, D152, D156, D157, D158, D159, D160, D161, D162, D163, D164, D165, D166, D167, D168, D169, D170, D171, D172, D173, D177, D178, D179, D180, D181, D183, D184, D186, D187, D188, D189, D190, D191, D192, D193, D194, D195, D196, D197, D198, D55, D75, D76, D77, D78, D79, D86, D87, D88, D89, D90, D91, D92, D93, D94, D95, D96, D97: footprint Diode_THT:D_DO-35_SOD27_P10.16mm_Horizontal -> sk6812 mini-e:D_DO-35_SOD27_P10.16mm_Horizontal
- MX1, MX10, MX11, MX12, MX13, MX14, MX15, MX16, MX17, MX18, MX19, MX2, MX20, MX21, MX22, MX23, MX24, MX25, MX26, MX27, MX28, MX29, MX3, MX30, MX31, MX32, MX33, MX34, MX35, MX36, MX37, MX38, MX39, MX4, MX40, MX41, MX42, MX43, MX44, MX45, MX46, MX47, MX48, MX49, MX5, MX50, MX51, MX52, MX53, MX54, MX55, MX56, MX57, MX58, MX59, MX6, MX60, MX61, MX62, MX63, MX64, MX65, MX66, MX67, MX68, MX69, MX7, MX70, MX71, MX72, MX73, MX74, MX75, MX76, MX77, MX78, MX79, MX8, MX80, MX81, MX82, MX83, MX84, MX85, MX86, MX87, MX88, MX89, MX9, MX90, MX91, MX92: symbol MX_Alps_Hybrid:MX-NoLED -> PENIS-rescue:MX-NoLED-MX_Alps_Hybrid
- U2: symbol Power_Protection:USBLC6-2SC6 -> PENIS-rescue:USBLC6-2SC6-Power_Protection
Connections:
- net COL0: now also U1.10 (PA0); no longer U1.41 (PB5)
- net COL1: now also U1.11 (PA1); no longer U1.34 (PA13)
- net COL10: now also U1.20 (PB2); no longer U1.10 (PA0)
- net COL11: now also U1.21 (PB10); no longer U1.11 (PA1)
- net COL12: now also U1.22 (PB11); no longer U1.12 (PA2)
- net COL13: now also U1.25 (PB12); no longer U1.13 (PA3)
- net COL14: now also U1.26 (PB13); no longer U1.14 (PA4)
- net COL15: now also U1.27 (PB14); no longer U1.15 (PA5)
- net COL16: now also U1.34 (PA13); no longer U1.16 (PA6)
- net COL17: now also U1.37 (PA14); no longer U1.17 (PA7)
- net COL2: now also U1.12 (PA2); no longer U1.37 (PA14)
- net COL3: now also U1.13 (PA3); no longer U1.45 (PB8)
- net COL4: now also U1.14 (PA4); no longer U1.46 (PB9)
- net COL5: now also U1.15 (PA5); no longer U1.21 (PB10)
- net COL6: now also U1.16 (PA6); no longer U1.22 (PB11)
- net COL7: now also U1.17 (PA7); no longer U1.25 (PB12)
- net COL8: now also U1.18 (PB0); no longer U1.26 (PB13)
- net COL9: now also U1.19 (PB1); no longer U1.27 (PB14)
- net ROW0: now also U1.46 (PB9); no longer U1.18 (PB0)
- net ROW1: now also U1.45 (PB8); no longer U1.19 (PB1)
- net ROW2: now also U1.41 (PB5); no longer U1.20 (PB2)
- net ROW3: now also U1.40 (PB4); no longer U1.39 (PB3)
- net ROW4: now also U1.39 (PB3); no longer U1.40 (PB4)
- net WS2812C_2: no longer names the net of U1.29 (PA8)
- no-connect marks 13 -> 18
Other:
- note removed: "RGB Backlight"
