File: PENIS.kicad_pcb (KiCad board)
At the start: 2 copper layers, 389.5 x 155.3 mm, 395 parts, among them J2 Conn_01x04_Female, P1 USB_C_Plug, Q1 DTC123J, SW1 SW_Push, SW2 Rotary_Encoder_Switch, U1 STM32F072C8T6, U2 USBLC6-2SC6, U3 XC6206P332MR

Commit message: Mounting holes
Routing:
- net +5V: track 2879.9 -> 2880.8 mm
Other:
- outline, holes or cut-outs redrawn
